File: recruiting.kicad_sch (KiCad schematic)
At the start: 1 part

Commit message: Add files via upload
Parts:
- added BT?: Battery_Cell, symbol Device:Battery_Cell
- added D?: LED, symbol Device:LED
- added MES?: Ammeter_AC, symbol Device:Ammeter_AC
- added Q?: 2N2219, Package_TO_SOT_THT:TO-39-3, symbol Transistor_BJT:2N2219
- added R? (x3): R_US, symbol Device:R_US
- added R?: R_Shunt, symbol Device:R_Shunt
- added R?: R_Small_US, symbol Device:R_Small_US
Connections:
- new net: BT?.1 (+), MES?.2, R?.1
- new net: D?.2 (A), Q?.1 (E)
- new net: Q?.2 (B), R?.2
- new net: Q?.3 (C), R?.2
- new net: R?.1, R?.1, R?.2
- new net A: R?.1
- new net B: BT?.2 (-), D?.1 (K), MES?.1, R?.2, R?.4
- new net D: R?.1
Other:
- added sheet lm78 (untitled.kicad_sch)
- added sheet lm783.3 (lm783.kicad_sch)
- note added: "1,65 Ω"
- note added: "1,67 Ω"
- note added: "11-27 V"
- note added: "70 Ω"
- moved on the sheet: C1

Commit message: Add files via upload
Parts:
- removed C1: 1F, Capacitor_SMD:C_0805_2012Metric, symbol Device:C
- removed D?: LED, symbol Device:LED
- removed Q?: 2N2219, Package_TO_SOT_THT:TO-39-3, symbol Transistor_BJT:2N2219
- removed R? (x2): R_US, symbol Device:R_US
Connections:
- net D is gone; now on net B: R?.1
- net B: now also R?.2
Other:
- added sheet Led (Led.kicad_sch)
- note removed: "70 Ω"
